File: FT817-BT-JDY67.kicad_sch (KiCad schematic)
At the start: 34 parts, among them J1009 Mini-DIN-8PR, J1010 Mini-DIN-6PR, Q1 2N7002, Q2 TP0610, U1 JDY-67 Bluetooth Module, U2 LM1117MP-5.0

Commit message: Fixed 2N7002 Footprint
Parts:
- C1, C2: symbol FT81x-BT_DIGI-Adapter_Library:C_Polarized -> Library:C_Polarized
- C3, C4, C5, C6, C7, C8: symbol FT81x-BT_DIGI-Adapter_Library:C -> Library:C
- D1, D2: symbol FT81x-BT_DIGI-Adapter_Library:LED -> Library:LED
- H1, H2, H3: symbol FT81x-BT_DIGI-Adapter_Library:MountingHole_Pad -> Library:MountingHole_Pad
- J1009: symbol FT81x-BT_DIGI-Adapter_Library:Mini-DIN-8PR -> Library:Mini-DIN-8PR
- J1010: symbol FT81x-BT_DIGI-Adapter_Library:Mini-DIN-6PR -> Library:Mini-DIN-6PR
- L1, L2, L3: symbol FT81x-BT_DIGI-Adapter_Library:L_Ferrite -> Library:L_Ferrite
- Q1: symbol FT81x-BT_DIGI-Adapter_Library:NMOS -> Library:NMOS
- Q2: symbol FT81x-BT_DIGI-Adapter_Library:PMOS -> Library:PMOS
- R1, R10, R11, R12, R2, R3, R4, R5, R6, R7, R8, R9: symbol FT81x-BT_DIGI-Adapter_Library:R -> Library:R
- U1: symbol FT81x-BT_DIGI-Adapter_Library:JDY-67_Bluetooth_Module -> Library:JDY-67_Bluetooth_Module
- U2: symbol FT81x-BT_DIGI-Adapter_Library:LM1117MP-3.3 -> Library:LM1117MP-3.3
Connections:
- net GND: now also Q1.2 (S); no longer Q1.3 (S)
- net at C8.1, R11.1, R12.2: now also Q1.1 (G); no longer Q1.2 (G)
- net at Q2.2 (G), R10.1: now also Q1.3 (D); no longer Q1.1 (D)
Changed lines of the file:
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@@
     )
   )
-  (symbol (lib_id "FT81x-BT_DIGI-Adapter_Library:R") (at 196.85 119.38 270) (mirror x) (unit 1)
+  (symbol (lib_id "Library:R") (at 196.85 119.38 270) (mirror x) (unit 1)
     (in_bom yes) (on_board yes) (dnp no)
     (property "Reference" "R2" (at 196.85 119.38 90)
@@
     )
   )
-  (symbol (lib_id "FT81x-BT_DIGI-Adapter_Library:MountingHole_Pad") (at 44.45 158.75 0) (unit 1)
+  (symbol (lib_id "Library:MountingHole_Pad") (at 44.45 158.75 0) (unit 1)
     (in_bom yes) (on_board yes) (dnp no) (fields_autoplaced)
     (property "Reference" "H2" (at 46.99 156.845 0)
@@
     )
   )
-  (symbol (lib_id "FT81x-BT_DIGI-Adapter_Library:MountingHole_Pad") (at 44.45 143.51 0) (unit 1)
+  (symbol (lib_id "Library:MountingHole_Pad") (at 44.45 143.51 0) (unit 1)
     (in_bom yes) (on_board yes) (dnp no) (fields_autoplaced)
     (property "Reference" "H1" (at 46.99 141.605 0)
@@
     )
   )
-  (symbol (lib_id "FT81x-BT_DIGI-Adapter_Library:C") (at 151.13 76.2 0) (unit 1)
+  (symbol (lib_id "Library:C") (at 151.13 76.2 0) (unit 1)
     (in_bom yes) (on_board yes) (dnp no)
     (property "Reference" "C8" (at 157.48 76.2 90)
@@
     )
   )
-  (symbol (lib_id "FT81x-BT_DIGI-Adapter_Library:R") (at 143.51 76.2 0) (mirror y) (unit 1)
+  (symbol (lib_id "Library:R") (at 143.51 76.2 0) (mirror y) (unit 1)
     (in_bom yes) (on_board yes) (dnp no)
     (property "Reference" "R11" (at 138.43 76.2 90)
@@
     )
   )
-  (symbol (lib_id "FT81x-BT_DIGI-Adapter_Library:C") (at 236.22 129.54 90) (unit 1)
+  (symbol (lib_id "Library:C") (at 236.22 129.54 90) (unit 1)
     (in_bom yes) (on_board yes) (dnp no)
     (property "Reference" "C3" (at 236.22 123.19 90)
@@
     )
   )
-  (symbol (lib_id "FT81x-BT_DIGI-Adapter_Library:JDY-67_Bluetooth_Module") (at 151.13 101.6 0) (unit 1)
+  (symbol (lib_id "Library:JDY-67_Bluetooth_Module") (at 151.13 101.6 0) (unit 1)
     (in_bom yes) (on_board yes) (dnp no) (fields_autoplaced)
     (property "Reference" "U1" (at 162.56 97.79 0)
@@
     )
   )
-  (symbol (lib_id "FT81x-BT_DIGI-Adapter_Library:R") (at 133.35 71.12 90) (mirror x) (unit 1)
+  (symbol (lib_id "Library:R") (at 133.35 71.12 90) (mirror x) (unit 1)
     (in_bom yes) (on_board yes) (dnp no)
     (property "Reference" "R12" (at 133.35 76.2 90)
@@
     )
   )
-  (symbol (lib_id "FT81x-BT_DIGI-Adapter_Library:R") (at 154.94 60.96 270) (mirror x) (unit 1)
+  (symbol (lib_id "Library:R") (at 154.94 60.96 270) (mirror x) (unit 1)
     (in_bom yes) (on_board yes) (dnp no)
     (property "Reference" "R10" (at 154.94 55.88 90)
@@
     )
   )
-  (symbol (lib_id "FT81x-BT_DIGI-Adapter_Library:PMOS") (at 162.56 53.34 270) (mirror x) (unit 1)
+  (symbol (lib_id "Library:PMOS") (at 162.56 53.34 270) (mirror x) (unit 1)
     (in_bom yes) (on_board yes) (dnp no)
     (property "Reference" "Q2" (at 162.56 44.45 90)
@@
     )
   )
-  (symbol (lib_id "FT81x-BT_DIGI-Adapter_Library:R") (at 133.35 114.3 270) (mirror x) (unit 1)
+  (symbol (lib_id "Library:R") (at 133.35 114.3 270) (mirror x) (unit 1)
     (in_bom yes) (on_board yes) (dnp no)
     (property "Reference" "R4" (at 133.35 114.3 90)
@@
     )
   )
-  (symbol (lib_id "FT81x-BT_DIGI-Adapter_Library:R") (at 196.85 99.06 270) (mirror x) (unit 1)
+  (symbol (lib_id "Library:R") (at 196.85 99.06 270) (mirror x) (unit 1)
     (in_bom yes) (on_board yes) (dnp no)
     (property "Reference" "R7" (at 196.85 99.06 90)
@@
     )
   )
-  (symbol (lib_id "FT81x-BT_DIGI-Adapter_Library:C_Polarized") (at 226.06 63.5 0) (unit 1)
+  (symbol (lib_id "Library:C_Polarized") (at 226.06 63.5 0) (unit 1)
     (in_bom yes) (on_board yes) (dnp no) (fields_autoplaced)
     (property "Reference" "C2" (at 229.87 61.976 0)
@@
     )
   )
-  (symbol (lib_id "FT81x-BT_DIGI-Adapter_Library:R") (at 212.09 149.86 0) (mirror y) (unit 1)
+  (symbol (lib_id "Library:R") (at 212.09 149.86 0) (mirror y) (unit 1)
     (in_bom yes) (on_board yes) (dnp no)
     (property "Reference" "R9" (at 212.09 149.86 90)
@@
     )
   )
-  (symbol (lib_id "FT81x-BT_DIGI-Adapter_Library:R") (at 222.25 129.54 90) (unit 1)
+  (symbol (lib_id "Library:R") (at 222.25 129.54 90) (unit 1)
     (in_bom yes) (on_board yes) (dnp no) (fields_autoplaced)
     (property "Reference" "R8" (at 222.25 124.46 90)
@@
     )
   )
-  (symbol (lib_id "FT81x-BT_DIGI-Adapter_Library:NMOS") (at 160.02 71.12 0) (unit 1)
-    (in_bom yes) (on_board yes) (dnp no) (fields_autoplaced)
+  (symbol (lib_id "Library:NMOS") (at 160.02 71.12 0) (unit 1)
+    (in_bom yes) (on_board yes) (dnp no)
     (property "Reference" "Q1" (at 166.37 70.485 0)
       (effects (font (size 1.27 1.27)) (justify left))
@@
       (effects (font (size 1.27 1.27)) hide)
     )
-    (property "Sim.Pins" "1=D 2=G 3=S" (at 160.02 86.36 0)
+    (property "Sim.Pins" "1=G 2=S 3=D" (at 160.02 86.36 0)
       (effects (font (size 1.27 1.27)) hide)
     )
@@
     )
   )
-  (symbol (lib_id "FT81x-BT_DIGI-Adapter_Library:Mini-DIN-6PR") (at 53.34 53.34 0) (unit 1)
+  (symbol (lib_id "Library:Mini-DIN-6PR") (at 53.34 53.34 0) (unit 1)
     (in_bom yes) (on_board yes) (dnp no)
     (property "Reference" "J1010" (at 53.34 66.04 0)
@@
     )
   )
-  (symbol (lib_id "FT81x-BT_DIGI-Adapter_Library:LED") (at 209.55 109.22 0) (mirror y) (unit 1)
+  (symbol (lib_id "Library:LED") (at 209.55 109.22 0) (mirror y) (unit 1)
     (in_bom yes) (on_board yes) (dnp no)
     (property "Reference" "D1" (at 211.1375 104.14 0)
@@
     )
   )
-  (symbol (lib_id "FT81x-BT_DIGI-Adapter_Library:C_Polarized") (at 200.66 63.5 0) (unit 1)
+  (symbol (lib_id "Library:C_Polarized") (at 200.66 63.5 0) (unit 1)
     (in_bom yes) (on_board yes) (dnp no) (fields_autoplaced)
     (property "Reference" "C1" (at 204.47 61.976 0)
@@
     )
   )
-  (symbol (lib_id "FT81x-BT_DIGI-Adapter_Library:C") (at 196.85 149.86 90) (unit 1)
+  (symbol (lib_id "Library:C") (at 196.85 149.86 90) (unit 1)
     (in_bom yes) (on_board yes) (dnp no)
     (property "Reference" "C5" (at 196.85 143.51 90)
@@
     )
   )
-  (symbol (lib_id "FT81x-BT_DIGI-Adapter_Library:C") (at 196.85 139.7 90) (unit 1)
+  (symbol (lib_id "Library:C") (at 196.85 139.7 90) (unit 1)
     (in_bom yes) (on_board yes) (dnp no)
     (property "Reference" "C4" (at 196.85 133.35 90)
@@
     )
   )
-  (symbol (lib_id "FT81x-BT_DIGI-Adapter_Library:L_Ferrite") (at 120.65 114.3 90) (unit 1)
+  (symbol (lib_id "Library:L_Ferrite") (at 120.65 114.3 90) (unit 1)
     (in_bom yes) (on_board yes) (dnp no) (fields_autoplaced)
     (property "Reference" "L2" (at 120.65 109.22 90)
@@
     )
   )
-  (symbol (lib_id "FT81x-BT_DIGI-Adapter_Library:R") (at 207.01 129.54 0) (mirror y) (unit 1)
+  (symbol (lib_id "Library:R") (at 207.01 129.54 0) (mirror y) (unit 1)
     (in_bom yes) (on_board yes) (dnp no)
     (property "Reference" "R5" (at 207.01 129.54 90)
@@
     )
   )
-  (symbol (lib_id "FT81x-BT_DIGI-Adapter_Library:C") (at 185.42 63.5 0) (unit 1)
+  (symbol (lib_id "Library:C") (at 185.42 63.5 0) (unit 1)
     (in_bom yes) (on_board yes) (dnp no)
     (property "Reference" "C7" (at 191.77 63.5 90)
@@
     )
   )
-  (symbol (lib_id "FT81x-BT_DIGI-Adapter_Library:R") (at 133.35 106.68 270) (mirror x) (unit 1)
+  (symbol (lib_id "Library:R") (at 133.35 106.68 270) (mirror x) (unit 1)
     (in_bom yes) (on_board yes) (dnp no)
     (property "Reference" "R3" (at 133.35 106.68 90)
@@
     )
   )
-  (symbol (lib_id "FT81x-BT_DIGI-Adapter_Library:LED") (at 209.55 119.38 0) (mirror y) (unit 1)
+  (symbol (lib_id "Library:LED") (at 209.55 119.38 0) (mirror y) (unit 1)
     (in_bom yes) (on_board yes) (dnp no)
     (property "Reference" "D2" (at 211.1375 114.3 0)
@@
     )
   )
-  (symbol (lib_id "FT81x-BT_DIGI-Adapter_Library:L_Ferrite") (at 120.65 106.68 90) (unit 1)
+  (symbol (lib_id "Library:L_Ferrite") (at 120.65 106.68 90) (unit 1)
     (in_bom yes) (on_board yes) (dnp no) (fields_autoplaced)
     (property "Reference" "L1" (at 120.65 101.6 90)
@@
     )
   )
-  (symbol (lib_id "FT81x-BT_DIGI-Adapter_Library:L_Ferrite") (at 179.07 50.8 90) (unit 1)
+  (symbol (lib_id "Library:L_Ferrite") (at 179.07 50.8 90) (unit 1)
     (in_bom yes) (on_board yes) (dnp no) (fields_autoplaced)
     (property "Reference" "L3" (at 179.07 45.72 90)
@@
     )
   )
-  (symbol (lib_id "FT81x-BT_DIGI-Adapter_Library:LM1117MP-3.3") (at 213.36 50.8 0) (unit 1)
+  (symbol (lib_id "Library:LM1117MP-3.3") (at 213.36 50.8 0) (unit 1)
     (in_bom yes) (on_board yes) (dnp no) (fields_autoplaced)
     (property "Reference" "U2" (at 213.36 44.45 0)
@@
     )
   )
-  (symbol (lib_id "FT81x-BT_DIGI-Adapter_Library:Mini-DIN-8PR") (at 52.07 93.98 0) (unit 1)
+  (symbol (lib_id "Library:Mini-DIN-8PR") (at 52.07 93.98 0) (unit 1)
     (in_bom yes) (on_board yes) (dnp no)
     (property "Reference" "J1009" (at 49.53 106.68 0)
@@
     )
   )
-  (symbol (lib_id "FT81x-BT_DIGI-Adapter_Library:R") (at 190.5 50.8 270) (mirror x) (unit 1)
+  (symbol (lib_id "Library:R") (at 190.5 50.8 270) (mirror x) (unit 1)
     (in_bom yes) (on_board yes) (dnp no)
     (property "Reference" "R6" (at 190.5 45.72 90)
@@
     )
   )
-  (symbol (lib_id "FT81x-BT_DIGI-Adapter_Library:MountingHole_Pad") (at 44.45 176.53 0) (unit 1)
+  (symbol (lib_id "Library:MountingHole_Pad") (at 44.45 176.53 0) (unit 1)
     (in_bom yes) (on_board yes) (dnp no) (fields_autoplaced)
     (property "Reference" "H3" (at 46.99 174.625 0)
@@
     )
   )
-  (symbol (lib_id "FT81x-BT_DIGI-Adapter_Library:C") (at 138.43 142.24 0) (unit 1)
+  (symbol (lib_id "Library:C") (at 138.43 142.24 0) (unit 1)
     (in_bom yes) (on_board yes) (dnp no)
     (property "Reference" "C6" (at 144.78 142.24 90)
@@
     )
   )
-  (symbol (lib_id "FT81x-BT_DIGI-Adapter_Library:R") (at 196.85 109.22 270) (mirror x) (unit 1)
+  (symbol (lib_id "Library:R") (at 196.85 109.22 270) (mirror x) (unit 1)
     (in_bom yes) (on_board yes) (dnp no)
     (property "Reference" "R1" (at 196.85 109.22 90)
