File: FT817-BT-JDY67.kicad_pcb (KiCad board)
At the start: 2 copper layers, 93.3 x 33.7 mm, 23 parts, among them J1009 Mini-DIN-8PR, J1010 Mini-DIN-6PR, U1 JDY-67 Bluetooth Module, U2 LM1117MP-3.3

Commit message: update
Parts:
- removed D3: LED, LED_SMD:LED_0805_2012Metric
- removed R5: 1k, Resistor_SMD:R_0805_2012Metric
- added D4: 1N4735/6.2V, Diode_SMD:D_SMA, F.Cu at (172.6, 81.3)
- added L1: 100uH, Inductor_SMD:L_0805_2012Metric_Pad1.05x1.20mm_HandSolder, F.Cu at (153.6, 85.1)
- added L2: 100uH, Inductor_SMD:L_0805_2012Metric_Pad1.05x1.20mm_HandSolder, F.Cu at (153.6, 87.6)
- added R8: 10k, Resistor_SMD:R_0805_2012Metric, F.Cu at (152.4, 80.4)
- added RV1: 1k, Potentiometer_SMD:Potentiometer_Bourns_3314J_Vertical, F.Cu at (148.0, 80.6)
- added RV2: 1k, Potentiometer_SMD:Potentiometer_Bourns_3314J_Vertical, F.Cu at (135.3, 73.0)
- C3, C4, C5: value 100n -> 1uF
- R6: value 100R -> 50R
- moved U2 5.99 mm to (166.4, 90.8)
- moved C1 5.72 mm to (171.4, 85.1), turned to 180 degrees
- moved C2 3.81 mm to (159.4, 91.5)
- moved R4 3.81 mm to (148.9, 87.6)
- moved R3 3.73 mm to (148.9, 85.1)
- moved C3 3.14 mm to (154.9, 80.3), turned to 90 degrees
- moved D1 2.54 mm to (126.4, 72.7)
- moved D2 2.54 mm to (128.9, 72.7)
- moved R6 1.91 mm to (174.6, 76.8)
Connections:
- C3 pad 1: Net-(U1-MIC-P) -> Net-(C3-Pad1)
- C4 pad 2: DATA IN -> Net-(C4-Pad2)
- C5 pad 2: DATA IN -> Net-(C4-Pad2)
- R3 pad 2: RX D -> Net-(L1-Pad2)
- R4 pad 2: TX D -> Net-(L2-Pad2)
Routing:
- net Net-(U1-RXD): track 52.3 -> 26.6 mm
- net Net-(C4-Pad2): track 0.00 -> 8.75 mm
- net 3.3V: track 33.2 -> 24.8 mm
- net Net-(D4-K): track 5.44 -> 13.4 mm
- net GND: track 11.8 -> 19.2 mm, vias 114 -> 111
- net Net-(U1-MIC-P): track 23.7 -> 18.7 mm
- net Net-(U1-TXD): track 33.7 -> 30.0 mm
- net DATA OUT 1200bps: track 24.5 -> 20.8 mm
- net DATA IN: track 34.1 -> 30.5 mm
- net Net-(L2-Pad2): track 0.00 -> 2.54 mm
- net Net-(L1-Pad2): track 0.00 -> 2.54 mm
- net Net-(C3-Pad1): track 0.00 -> 2.54 mm
- net Net-(D3-A): track 2.49 -> 0.00 mm
- net Net-(R8-Pad1): track 0.00 -> 2.31 mm
- net TX D: track 31.9 -> 30.8 mm
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Other:
- board text added: "MIC"
- board text added: "OUT"
- board text added: "© BG6LH v20230522"
- board text removed: "TXD"
- board text removed: "© BG6LH v20230517"

Commit message: minimal update
Parts:
- R3, R4: value 22 -> 22R
- R6: value 50R -> 51R
Connections:
- J1009 pad : GND -> (no net)
- J1010 pad : GND -> (no net)
Other:
- board text added: "A.RX"
- board text added: "A.TX"
- board text removed: "MIC"
- board text removed: "OUT"
Changed lines of the file:
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@@
   (title_block
     (title "FT-81x BT DIGI Adaptor")
-    (date "2023-05-17")
-    (rev "20230517")
-    (company "BG6LH")
+    (date "2023-05-22")
+    (rev "20230522")
+    (company "https://github.com/BG6LH/FT-81x-BT-DIGI-Adaptor")
     (comment 1 "CC-BY-NC-SA 4.0")
     (comment 2 "With special thanks to: BG6JJI, BI1EIH")
@@
     (fp_circle (center 0 0) (end 4.5 0)
       (stroke (width 0.127) (type default)) (fill none) (layer "F.Fab"))
-    (pad "" thru_hole oval (at 0 -4.4) (size 4 1.8) (drill oval 3.2 0.8) (layers "*.Cu" "*.Mask")
-      (net 24 "GND"))
+    (pad "" thru_hole oval (at 0 -4.4) (size 4 1.8) (drill oval 3.2 0.8) (layers "*.Cu" "*.Mask"))
     (pad "1" thru_hole rect (at 1 2.4) (size 1.6 1.3) (drill oval 1.2 0.9) (layers "*.Cu" "*.Mask")
       (net 10 "+13.8V") (pintype "passive"))
@@
         (effects (font (size 1 1) (thickness 0.15)))
     )
-    (fp_text value "22" (at 0 1.65) (layer "F.Fab") hide
+    (fp_text value "22R" (at 0 1.65) (layer "F.Fab") hide
         (effects (font (size 1 1) (thickness 0.15)))
     )
@@
     (fp_line (start 1 0.625) (end -1 0.625)
       (stroke (width 0.1) (type solid)) (layer "F.Fab"))
-    (pad "1" smd roundrect (at -0.9125 0 270) (size 1.025 1.4) (layers "F.Cu" "F.Paste" "F.Mask") (roundrect_rratio 0.243902)
+    (pad "1" smd roundrect (at -0.9125 0 270) (size 1.025 1.4) (layers "F.Cu" "F.Paste" "F.Mask") (roundrect_rratio 0.243902439)
       (net 38 "Net-(R8-Pad1)") (pintype "passive"))
-    (pad "2" smd roundrect (at 0.9125 0 270) (size 1.025 1.4) (layers "F.Cu" "F.Paste" "F.Mask") (roundrect_rratio 0.243902)
+    (pad "2" smd roundrect (at 0.9125 0 270) (size 1.025 1.4) (layers "F.Cu" "F.Paste" "F.Mask") (roundrect_rratio 0.243902439)
       (net 34 "Net-(C3-Pad1)") (pintype "passive"))
     (model "${KICAD6_3DMODEL_DIR}/Resistor_SMD.3dshapes/R_0805_2012Metric.wrl"
@@
         (effects (font (size 1 1) (thickness 0.15)))
     )
-    (fp_text value "22" (at 0 1.65) (layer "F.Fab") hide
+    (fp_text value "22R" (at 0 1.65) (layer "F.Fab") hide
         (effects (font (size 1 1) (thickness 0.15)))
     )
@@
         (effects (font (size 1 1) (thickness 0.15)))
     )
-    (fp_text value "50R" (at 0 1.65 90) (layer "F.Fab") hide
+    (fp_text value "51R" (at 0 1.65 90) (layer "F.Fab") hide
         (effects (font (size 1 1) (thickness 0.15)))
     )
@@
     (fp_line (start 1 0.45) (end -1 0.45)
       (stroke (width 0.1) (type solid)) (layer "F.Fab"))
-    (pad "1" smd roundrect (at -1.15 0 180) (size 1.05 1.2) (layers "F.Cu" "F.Paste" "F.Mask") (roundrect_rratio 0.238095)
+    (pad "1" smd roundrect (at -1.15 0 180) (size 1.05 1.2) (layers "F.Cu" "F.Paste" "F.Mask") (roundrect_rratio 0.2380952381)
       (net 12 "TX D") (pinfunction "1") (pintype "passive"))
-    (pad "2" smd roundrect (at 1.15 0 180) (size 1.05 1.2) (layers "F.Cu" "F.Paste" "F.Mask") (roundrect_rratio 0.238095)
+    (pad "2" smd roundrect (at 1.15 0 180) (size 1.05 1.2) (layers "F.Cu" "F.Paste" "F.Mask") (roundrect_rratio 0.2380952381)
       (net 37 "Net-(L2-Pad2)") (pinfunction "2") (pintype "passive"))
     (model "${KICAD6_3DMODEL_DIR}/Inductor_SMD.3dshapes/L_0805_2012Metric.wrl"
@@
     (fp_circle (center 0 0) (end 4.5 0)
       (stroke (width 0.127) (type default)) (fill none) (layer "F.Fab"))
-    (pad "" thru_hole oval (at 0 -4.4) (size 4 1.8) (drill oval 3.2 0.8) (layers "*.Cu" "*.Mask")
-      (net 24 "GND"))
+    (pad "" thru_hole oval (at 0 -4.4) (size 4 1.8) (drill oval 3.2 0.8) (layers "*.Cu" "*.Mask"))
     (pad "1" thru_hole rect (at 1 2.4) (size 1.6 1.3) (drill oval 1.2 0.9) (layers "*.Cu" "*.Mask")
       (net 18 "DATA IN") (pintype "passive"))
@@
     (fp_line (start 1 0.45) (end -1 0.45)
       (stroke (width 0.1) (type solid)) (layer "F.Fab"))
-    (pad "1" smd roundrect (at -1.15 0 180) (size 1.05 1.2) (layers "F.Cu" "F.Paste" "F.Mask") (roundrect_rratio 0.238095)
+    (pad "1" smd roundrect (at -1.15 0 180) (size 1.05 1.2) (layers "F.Cu" "F.Paste" "F.Mask") (roundrect_rratio 0.2380952381)
       (net 13 "RX D") (pinfunction "1") (pintype "passive"))
-    (pad "2" smd roundrect (at 1.15 0 180) (size 1.05 1.2) (layers "F.Cu" "F.Paste" "F.Mask") (roundrect_rratio 0.238095)
+    (pad "2" smd roundrect (at 1.15 0 180) (size 1.05 1.2) (layers "F.Cu" "F.Paste" "F.Mask") (roundrect_rratio 0.2380952381)
       (net 36 "Net-(L1-Pad2)") (pinfunction "2") (pintype "passive"))
     (model "${KICAD6_3DMODEL_DIR}/Inductor_SMD.3dshapes/L_0805_2012Metric.wrl"
@@
   (gr_arc (start 154.305 64.77) (mid 154.862962 63.422962) (end 156.21 62.865)
     (stroke (width 0.1) (type default)) (layer "Edge.Cuts"))
-  (image (at 143.51 79.375) (layer "User.2") (scale 0.229514)
+  (image (at 143.51 80.01) (layer "User.2") (scale 0.229514)
     (data
       iVBORw0KGgoAAAANSUhEUgAADOQAAAOgCAIAAACoDt/6AAAAA3NCSVQICAjb4U/gAAAACXBIWXMA
@@
     )
   )
-  (image (at 143.51 80.01) (layer "User.2") (scale 0.229514)
+  (image (at 143.51 79.375) (layer "User.2") (scale 0.229514)
     (data
       iVBORw0KGgoAAAANSUhEUgAADOQAAAOgCAIAAACoDt/6AAAAA3NCSVQICAjb4U/gAAAACXBIWXMA
@@
     (effects (font (size 1 1) (thickness 0.15)) (justify left))
   )
-  (gr_text "OUT" (at 137.16 69.85) (layer "F.SilkS")
+  (gr_text "A.TX" (at 136.525 69.85) (layer "F.SilkS")
     (effects (font (size 1 1) (thickness 0.15)))
   )
@@
     (effects (font (size 0.8 0.8) (thickness 0.1)) (justify right))
   )
-  (gr_text "MIC" (at 149.225 77.47) (layer "F.SilkS")
+  (gr_text "A.RX" (at 149.225 77.47) (layer "F.SilkS")
     (effects (font (size 1 1) (thickness 0.15)))
   )

Commit message: update
Parts:
- H3: footprint BG6LH_Kicad_Libary:FT-817_GND_terminal_8.4mm_M8_Pad_TopBottom -> FT81x-BT-DIGI-Adapter-Library:FT-817_GND_terminal_8.4mm_M8_Pad_TopBottom
- J1009: footprint BG6LH_MiniDin_Pin:MD-8Pin -> FT81x-BT-DIGI-Adapter-Library:MD-8Pin_Reverse
- J1010: footprint BG6LH_MiniDin_Pin:MD-6Pin -> FT81x-BT-DIGI-Adapter-Library:MD-6Pin_Reverse
- R6: value 51R -> 270R
- U1: footprint BG6LH_Kicad_Libary:JDY-67_Bluetooth_Module -> FT81x-BT-DIGI-Adapter-Library:JDY-67_Bluetooth_Module
Other:
- board text added: "© BG6LH v20230527"
- board text removed: "© BG6LH v20230522"

Commit message: update
Parts:
- removed D4: 1N4735/6.2V, Diode_SMD:D_SMA
- removed RV1, RV2: 1k, Potentiometer_SMD:Potentiometer_Bourns_3314J_Vertical
- added C7: 100n, Capacitor_SMD:C_0805_2012Metric, F.Cu at (170.5, 80.0)
- added C8: 100n, Capacitor_SMD:C_0805_2012Metric, F.Cu at (166.4, 75.6)
- added L3: 100uH, Inductor_SMD:L_0805_2012Metric_Pad1.05x1.20mm_HandSolder, F.Cu at (173.4, 81.3)
- added Q1: 2N7002, Package_TO_SOT_SMD:SOT-23-3, F.Cu at (170.5, 77.0)
- added Q2: TP0610, Package_TO_SOT_SMD:SOT-23-3, F.Cu at (174.3, 77.0)
- added R10: 10k, Resistor_SMD:R_0805_2012Metric, F.Cu at (177.2, 76.8)
- added R11: 10k, Resistor_SMD:R_0805_2012Metric, F.Cu at (170.8, 72.7)
- added R12: 10k, Resistor_SMD:R_0805_2012Metric, F.Cu at (168.9, 72.7)
- added R5: 1k, Resistor_SMD:R_0805_2012Metric, F.Cu at (148.0, 81.6)
- added R9: 1k, Resistor_SMD:R_0805_2012Metric, F.Cu at (135.3, 75.9)
- R6: value 270R -> 150R
- U2: value LM1117MP-3.3 -> LM1117MP-5.0
- moved R6 7.03 mm to (170.5, 82.5), turned to 0 degrees
- moved C3 2.29 mm to (153.0, 81.6), turned to -90 degrees
- moved R8 2.29 mm to (150.5, 81.6), turned to 90 degrees
- moved C1 0.63 mm to (170.7, 85.1), turned to 0 degrees
Connections:
- net 3.3V renamed 5V
- C4 pad 2: Net-(C4-Pad2) -> DATA IN
- C5 pad 2: Net-(C4-Pad2) -> DATA IN
- R6 pad 2: +13.8V -> Net-(C7-Pad1)
- R8 pad 1: Net-(R8-Pad1) -> Net-(U1-MIC-P)
Routing:
- net Net-(Q1-D): track 0.00 -> 13.5 mm, vias 0 -> 2
- net GND: track 19.2 -> 8.85 mm, vias 111 -> 86
- net Net-(Q1-G): track 0.00 -> 9.55 mm
- net Net-(C4-Pad2): track 8.75 -> 0.00 mm
- net Net-(U2-VI): track 13.4 -> 5.42 mm
- net PTT: track 0.00 -> 6.20 mm, vias 0 -> 1
- net DATA IN: track 30.5 -> 36.7 mm, vias 1 -> 0
- net Net-(C7-Pad1): track 0.00 -> 4.32 mm
- net Net-(U1-MIC-P): track 18.7 -> 22.4 mm, vias 2 -> 0
- net Net-(R8-Pad1): track 2.31 -> 0.00 mm
- net Net-(Q2-D): track 0.00 -> 2.02 mm
- net +13.8V: track 7.21 -> 8.23 mm
- net DATA OUT 1200bps: track 20.8 -> 21.5 mm, vias 1 -> 0
Other:
- board text added: "© BG6LH v20230608"
- board text removed: "A.RX"
- board text removed: "A.TX"
- board text removed: "© BG6LH v20230527"

Commit message: Important update
Parts:
- H3: footprint FT81x-BT-DIGI-Adapter-Library:FT-817_GND_terminal_8.4mm_M8_Pad_TopBottom -> Library:FT-817_GND_terminal_8.4mm_M8_Pad_TopBottom
- J1009: footprint FT81x-BT-DIGI-Adapter-Library:MD-8Pin_Reverse -> Library:MD-8Pin_Reverse
- J1010: footprint FT81x-BT-DIGI-Adapter-Library:MD-6Pin_Reverse -> Library:MD-6Pin_Reverse
- Q1: footprint Package_TO_SOT_SMD:SOT-23-3 -> Package_TO_SOT_SMD:SOT-23
- Q2: value TP0610 -> TP0610T; footprint Package_TO_SOT_SMD:SOT-23-3 -> Package_TO_SOT_SMD:SOT-23
- U1: footprint FT81x-BT-DIGI-Adapter-Library:JDY-67_Bluetooth_Module -> Library:JDY-67_Bluetooth_Module
- moved Q1 1.27 mm to (169.2, 77.2), turned to 0 degrees
- moved L3 0.75 mm to (173.4, 82.0)
- moved C8 0.71 mm to (165.7, 75.9)
- moved Q2 0.65 mm to (173.7, 77.2), turned to 180 degrees
- moved R11 0.64 mm to (170.8, 72.1)
- moved R12 0.64 mm to (168.9, 72.1)
- moved R6 0.64 mm to (170.5, 83.2)
- moved C1 0.63 mm to (170.7, 85.7)
- moved C7 0.63 mm to (170.5, 80.6)
- moved R10 0.36 mm to (177.2, 77.2)
Connections:
- Q1 pad 1: Net-(Q1-D) -> Net-(Q1-G)
- Q1 pad 2: Net-(Q1-G) -> GND
- Q1 pad 3: GND -> Net-(Q1-D)
- Q2 pad 1: Net-(Q2-D) -> Net-(Q1-D)
- Q2 pad 2: Net-(Q1-D) -> +13.8V
- Q2 pad 3: +13.8V -> Net-(Q2-D)
Routing:
- net Net-(Q1-D): track 13.5 -> 8.48 mm, vias 2 -> 0
- net Net-(Q2-D): track 2.02 -> 3.98 mm
- net Net-(Q1-G): track 9.55 -> 8.43 mm
- net PTT: track 6.20 -> 5.14 mm
- net DATA OUT 1200bps: track 21.5 -> 22.6 mm
- net +13.8V: track 8.23 -> 7.40 mm
- net GND: track 8.85 -> 8.22 mm, vias 86 -> 88
- net Net-(U2-VI): track 5.42 -> 4.78 mm
- net Net-(C7-Pad1): track 4.32 -> 3.81 mm
Other:
- board text added: "© BG6LH v20230609"
- board text removed: "© BG6LH v20230608"
