File: FT817-BT-JDY67.kicad_pcb (KiCad board)
At the start: 2 copper layers, 93.3 x 33.7 mm, 34 parts, among them J1009 Mini-DIN-8PR, J1010 Mini-DIN-6PR, Q1 2N7002, Q2 TP0610T, U1 JDY-67 Bluetooth Module, U2 LM1117MP-5.0

Commit message: resistors value update
updated power supply's resistor right value.
Parts:
- R10, R11: value 10k -> 100k
- R12: value 10k -> 1k
- R6: value 150R -> 10R
- U2: value LM1117MP-5.0 -> LM1117MP-3.3
Changed lines of the file:
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@@
         (effects (font (size 1 1) (thickness 0.15)))
     )
-    (fp_text value "10k" (at 0 1.65 90) (layer "F.Fab") hide
+    (fp_text value "100k" (at 0 1.65 90) (layer "F.Fab") hide
         (effects (font (size 1 1) (thickness 0.15)))
     )
@@
         (effects (font (size 1 1) (thickness 0.15)))
     )
-    (fp_text value "150R" (at 0 1.65) (layer "F.Fab") hide
+    (fp_text value "10R" (at 0 1.65) (layer "F.Fab") hide
         (effects (font (size 1 1) (thickness 0.15)))
     )
@@
         (effects (font (size 1 1) (thickness 0.15)))
     )
-    (fp_text value "10k" (at 0 1.65 90) (layer "F.Fab") hide
+    (fp_text value "100k" (at 0 1.65 90) (layer "F.Fab") hide
         (effects (font (size 1 1) (thickness 0.15)))
     )
@@
         (effects (font (size 1 1) (thickness 0.15)))
     )
-    (fp_text value "LM1117MP-5.0" (at 0 4.5 180) (layer "F.Fab") hide
+    (fp_text value "LM1117MP-3.3" (at 0 4.5 180) (layer "F.Fab") hide
         (effects (font (size 1 1) (thickness 0.15)))
     )
@@
         (effects (font (size 1 1) (thickness 0.15)))
     )
-    (fp_text value "10k" (at 0 1.65 -90) (layer "F.Fab") hide
+    (fp_text value "1k" (at 0 1.65 -90) (layer "F.Fab") hide
         (effects (font (size 1 1) (thickness 0.15)))
     )
@@
   (gr_arc (start 154.305 64.77) (mid 154.862962 63.422962) (end 156.21 62.865)
     (stroke (width 0.1) (type default)) (layer "Edge.Cuts"))
-  (image (at 143.51 80.01) (layer "User.2") (scale 0.229514)
+  (image (at 143.51 79.375) (layer "User.2") (scale 0.229514)
     (data
       iVBORw0KGgoAAAANSUhEUgAADOQAAAOgCAIAAACoDt/6AAAAA3NCSVQICAjb4U/gAAAACXBIWXMA
@@
     )
   )
-  (image (at 143.51 79.375) (layer "User.2") (scale 0.229514)
+  (image (at 143.51 80.01) (layer "User.2") (scale 0.229514)
     (data
       iVBORw0KGgoAAAANSUhEUgAADOQAAAOgCAIAAACoDt/6AAAAA3NCSVQICAjb4U/gAAAACXBIWXMA
